File: cellyjamjam_v2.sch (EAGLE design)
At the start: 42 parts, among them IC4 LM1458, Q2 MMBT3904

Commit message: designin'
Parts:
- added OUTPUT: out, SparkFun-Connectors:M02LOCK_LONGPADS
- added POWER/GND, POWER/GND2: M02LOCK_LONGPADS, SparkFun-Connectors:M02LOCK_LONGPADS
- NOISEAMP, SWEEPAMP: value 5K/10TURN -> 5K
- VCOOFFSET: value 5K/10TURN -> 5k
Connections:
- new net N$33: C11.2, POWER/GND2.1, R17.2, R19.1
- net GND: now also OUTPUT.2, POWER/GND.2, POWER/GND2.2, VCOOFFSET.1; no longer VCOOFFSET.3
- net N$52: now also OUTPUT.1
- net VCC: now also POWER/GND.1, VCOOFFSET.3; no longer C11.2, R17.2, R19.1, VCOOFFSET.1
Other:
- moved on the sheet: C14, C22, D2, R20, R8, VCOOFFSET

Commit message: fuuuuuuu had to hand draw the ulp
Parts:
- C19: device SparkFun-Capacitors:CAP_POLC -> SparkFun-Capacitors:CAP_POLPTH1
- C21: device SparkFun-Capacitors:CAP_POLC -> SparkFun-Capacitors:CAP_POLPTH2
- C23: device SparkFun-Capacitors:CAP_POLD -> SparkFun-Capacitors:CAP_POLPTH1
- NOISEGEN: value LM386M-1 -> LM386N-1; device linear:LM386M-1 -> linear:LM386N-1
- ZENDIODE: device zetex:DSOD323 -> SparkFun-DiscreteSemi:DIODE-ZENERPTH
Other:
- note added: "cellyjamjamv2 allison burtch 30 april 2014"
- note removed: "Cellyjam_v1 Allison Burtch April 2014"
Changed lines of the file:
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@@
 <parts>
 <part name="VOLTAGEINVERT" library="maxim" deviceset="ICL7660CSA" device=""/>
-<part name="NOISEGEN" library="linear" deviceset="LM386?-*" device="M" technology="1"/>
+<part name="NOISEGEN" library="linear" deviceset="LM386?-*" device="N" technology="1" value="LM386N-1"/>
 <part name="GND1" library="supply0" deviceset="GND" device=""/>
 <part name="GND2" library="supply0" deviceset="GND" device=""/>
@@
 <part name="C17" library="SparkFun-Capacitors" deviceset="CAP_POL" device="C" value="10uF"/>
 <part name="C18" library="SparkFun-Capacitors" deviceset="CAP_POL" device="C" value="10uF"/>
-<part name="C19" library="SparkFun-Capacitors" deviceset="CAP_POL" device="C" value="10uF"/>
-<part name="C21" library="SparkFun-Capacitors" deviceset="CAP_POL" device="C" value="10uF"/>
+<part name="C19" library="SparkFun-Capacitors" deviceset="CAP_POL" device="PTH1" value="10uF"/>
+<part name="C21" library="SparkFun-Capacitors" deviceset="CAP_POL" device="PTH2" value="10uF"/>
 <part name="GND8" library="supply0" deviceset="GND" device=""/>
 <part name="R23" library="SparkFun-Resistors" deviceset="RESISTOR" device="0603-RES" value="100k"/>
@@
 <part name="GND13" library="supply0" deviceset="GND" device=""/>
 <part name="GND14" library="supply0" deviceset="GND" device=""/>
-<part name="C23" library="SparkFun-Capacitors" deviceset="CAP_POL" device="D" value="100uF"/>
+<part name="C23" library="SparkFun-Capacitors" deviceset="CAP_POL" device="PTH1" value="100uF"/>
 <part name="GND15" library="supply0" deviceset="GND" device=""/>
 <part name="GND16" library="supply0" deviceset="GND" device=""/>
@@
 <part name="GND26" library="supply0" deviceset="GND" device=""/>
 <part name="Q2" library="transistor-npn" deviceset="MMBT3904*" device=""/>
-<part name="ZENDIODE" library="zetex" deviceset="D" device="SOD323" value="MMBZ5235BW"/>
+<part name="ZENDIODE" library="SparkFun-DiscreteSemi" deviceset="DIODE-ZENER" device="PTH" value="MMBZ5235BW"/>
 <part name="D2" library="zetex" deviceset="D" device="SOD323" value="1N4148"/>
 <part name="JFET" library="transistor-fet" deviceset="MMBF5484*" device="" value="MMBF5484*"/>
@@
 <sheet>
 <plain>
-<text x="224.79" y="-25.4" size="1.778" layer="94">Cellyjam_v1
-Allison Burtch
-April 2014</text>
+<text x="205.74" y="-20.32" size="1.778" layer="91">cellyjamjamv2
+allison burtch
+30 april 2014</text>
 </plain>
 <instances>
